File: CurrentLimiter2.kicad_sch (KiCad schematic)
At the start: 10 parts, among them J1 Screw_Terminal_01x02, J2 Screw_Terminal_01x02, Q1 BCP54, Q2 MJD112

Commit message: v2 wersja wyslana do Elpinu do wykonania i zmontowania w Blaberk
Parts:
- removed JP1: SolderJumper_2_Open, Jumper:SolderJumper-2_P1.3mm_Open_RoundedPad1.0x1.5mm, symbol Jumper:SolderJumper_2_Open
- removed R4: R, Resistor_SMD:R_1206_3216Metric_Pad1.30x1.75mm_HandSolder, symbol Device:R
- Q2: footprint Package_TO_SOT_SMD:TO-263-2 -> Package_TO_SOT_SMD:TO-252-3_TabPin2
- R1: value 5k -> 7k15
- R2: value R -> 20m
- R3: value R -> 470m; footprint Resistor_SMD:R_1206_3216Metric_Pad1.30x1.75mm_HandSolder -> Resistor_SMD:R_2010_5025Metric_Pad1.40x2.65mm_HandSolder
Connections:
- net at J1.2 (Pin_2), R3.2: now also Q1.3 (B); no longer Q1.1 (E), R2.2
- net at Q2.3 (E): now also Q1.1 (E), R2.1; no longer Q1.3 (B)
- net at R3.1: now also R2.2; no longer R2.1
Other:
- moved on the sheet: Q1, R3

Commit message: zmieniona podstawka Darlingtona na 2 pinowa
Parts:
- Q2: footprint Package_TO_SOT_SMD:TO-252-3_TabPin2 -> Package_TO_SOT_SMD:TO-252-2
Changed lines of the file:
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@@
 			)
 		)
-		(property "Footprint" "Package_TO_SOT_SMD:TO-252-3_TabPin2"
+		(property "Footprint" "Package_TO_SOT_SMD:TO-252-2"
 			(at 142.24 102.235 0)
 			(effects
